Commit message: Added modifications to work with ws monitoring and marker estimation

File: hector_sensors_description/urdf/asus_camera.urdf.xacro (robot description, xacro)
@@ -65,37 +65,37 @@
     </xacro:macro>
     <!--
-     The asus_camera macro only adds the model, and also adds
-     the openni gazebo plugin.
-    -->
-    <xacro:macro name="asus_camera" params="name parent *origin">
-      <xacro:asus_camera_model name="${name}" parent="${parent}">
-        <xacro:insert_block name="origin" />
-      </xacro:asus_camera_model>
-      <!-- ASUS Xtion PRO camera for simulation -->
-      <gazebo reference="${name}_depth_frame">
-        <sensor type="depth" name="${name}">
-          <update_rate>20</update_rate>
-          <camera>
-            <horizontal_fov>${62.8 * M_PI/180.0}</horizontal_fov>
-            <image>
-              <format>R8G8B8</format>
-              <width>640</width>
-              <height>480</height>
-            </image>
-            <clip>
-              <near>0.5</near>
-              <far>9</far>
-            </clip>
-          </camera>
-          <plugin name="${name}_camera_controller" filename="libgazebo_ros_openni_kinect.so">
-            <imageTopicName>${name}/rgb/image_raw</imageTopicName>
-            <cameraInfoTopicName>${name}/rgb/camera_info</cameraInfoTopicName>
-            <depthImageTopicName>${name}/depth/image_raw</depthImageTopicName>
-            <depthImageCameraInfoTopicName>${name}/depth/camera_info</depthImageCameraInfoTopicName>
-            <pointCloudTopicName>${name}/depth/points</pointCloudTopicName>
-            <frameName>${name}_depth_optical_frame</frameName>
-          </plugin>
-        </sensor>
-      </gazebo>
-    </xacro:macro>
+    The asus_camera macro only adds the model, and also adds
+    the openni gazebo plugin.
+  -->
+  <xacro:macro name="asus_camera" params="name parent *origin min_range max_range">
+    <xacro:asus_camera_model name="${name}" parent="${parent}">
+      <xacro:insert_block name="origin" />
+    </xacro:asus_camera_model>
+    <!-- ASUS Xtion PRO camera for simulation -->
+    <gazebo reference="${name}_depth_frame">
+      <sensor type="depth" name="${name}">
+        <update_rate>20</update_rate>
+        <camera>
+          <horizontal_fov>${62.8 * M_PI/180.0}</horizontal_fov>
+          <image>
+            <format>R8G8B8</format>
+            <width>800</width>
+            <height>600</height>
+          </image>
+          <clip>
+            <near>${min_range}</near>
+            <far>${max_range}</far>
+          </clip>
+        </camera>
+        <plugin name="${name}_camera_controller" filename="libgazebo_ros_openni_kinect.so">
+          <imageTopicName>${name}/rgb/image_raw</imageTopicName>
+          <cameraInfoTopicName>${name}/rgb/camera_info</cameraInfoTopicName>
+          <depthImageTopicName>${name}/depth/image_raw</depthImageTopicName>
+          <depthImageCameraInfoTopicName>${name}/depth/camera_info</depthImageCameraInfoTopicName>
+          <pointCloudTopicName>${name}/depth/points</pointCloudTopicName>
+          <frameName>${name}_depth_optical_frame</frameName>
+        </plugin>
+      </sensor>
+    </gazebo>
+  </xacro:macro>
   </robot>
